Commit message: Add rplidar

File: description/urdf/diffbot.urdf.xacro (robot description, xacro)
@@ -4,4 +4,5 @@
   <xacro:arg name="prefix" default="" />
   <xacro:include filename="$(find diffdrive_arduino)/urdf/diffbot_description.urdf.xacro" />
+  <xacro:include filename="$(find diffdrive_arduino)/urdf/lidar.xacro" />
   <!-- Import Rviz colors -->
   <xacro:include filename="$(find diffdrive_arduino)/urdf/diffbot.materials.xacro" />

File: description/urdf/diffbot_description.urdf.xacro (robot description, xacro)
@@ -1,4 +1,5 @@
 <?xml version="1.0"?>
 <robot xmlns:xacro="http://www.ros.org/wiki/xacro">
+  <xacro:include filename="inertial_macros.xacro"/>
   <xacro:macro name="diffbot" params="prefix">
   <!-- Constants for robot dimensions -->
@@ -100,33 +101,4 @@
         </inertial>
       </link>
-    <joint name="${prefix}caster_frontal_wheel_joint" type="fixed">
-      <parent link="${prefix}base_link"/>
-      <child link="${prefix}caster_frontal_wheel"/>
-      <origin xyz="${base_width/2 - caster_wheel_radius} 0 ${z_offset}" rpy="0 0 0"/>
-    </joint>
-    <!-- caster frontal wheel Link -->
-    <link name="${prefix}caster_frontal_wheel">
-      <collision>
-        <origin xyz="0 0 0" rpy="0 0 0"/>
-        <geometry>
-          <sphere radius="${caster_wheel_radius}"/>
-        </geometry>
-      </collision>
-      <visual>
-        <origin xyz="0 0 0" rpy="0 0 0"/>
-        <geometry>
-          <sphere radius="${caster_wheel_radius}"/>
-        </geometry>
-        <material name="white"/>
-      </visual>
-      <inertial>
-        <origin xyz="0 0 0" rpy="0 0 0"/>
-        <mass value="${caster_wheel_mass}"/>
-        <inertia
-          ixx="${caster_wheel_mass * 0.4 * (caster_wheel_radius * caster_wheel_radius)}" ixy="0.0" ixz="0.0"
-          iyy="${caster_wheel_mass * 0.4 * (caster_wheel_radius * caster_wheel_radius)}" iyz="0.0"
-          izz="${caster_wheel_mass * 0.4 * (caster_wheel_radius * caster_wheel_radius)}"/>
-        </inertial>
-      </link>
     <joint name="${prefix}caster_rear_wheel_joint" type="fixed">
       <parent link="${prefix}base_link"/>
