Commit message: fix urdf

File: description/urdf/diffbot_description.urdf.xacro (robot description, xacro)
@@ -13,5 +13,5 @@
   <xacro:property name="wheel_radius" value="0.0475" />
   <xacro:property name="wheel_xoff" value="0.054"/>
-  <xacro:property name="wheel_zoff" value="-0.005"/>
+  <xacro:property name="wheel_zoff" value="0.03"/>
   <xacro:property name="caster_wheel_mass" value="0.1" /> <!-- arbitrary value for caster wheel mass -->
   <xacro:property name="caster_wheel_radius" value="0.015" />
@@ -106,5 +106,5 @@
       <parent link="${prefix}base_link"/>
       <child link="${prefix}caster_wheel"/>
-      <origin xyz="${caster_xoff} 0 ${-(base_height/2)}" rpy="0 0 0"/>
+      <origin xyz="${caster_xoff} 0 0" rpy="0 0 0"/>
     </joint>
     <!-- caster rear wheel Link -->

File: description/urdf/lidar.xacro (robot description, xacro)
@@ -4,5 +4,5 @@
         <parent link="base_link"/>
         <child link="laser_frame"/>
-        <origin xyz="0 0 0.12" rpy="0 0 0"/>
+        <origin xyz="0.054 0 0.12" rpy="0 0 0"/>
     </joint>
     <link name="laser_frame">
