Commit message: Setup URDF

File: description/ros2_control/diffbot.ros2_control.xacro (robot description, xacro)
@@ -11,5 +11,5 @@
         <param name="baud_rate">57600</param>
         <param name="timeout_ms">1000</param>
-        <param name="enc_counts_per_rev">3200</param>
+        <param name="enc_counts_per_rev">3200</param> <!-- 200 steps x 16 micro step = 3200 -->
         <param name="pid_p">20</param>
         <param name="pid_d">12</param>

File: description/urdf/diffbot.urdf.xacro (robot description, xacro)
@@ -10,5 +10,4 @@
   <xacro:include filename="$(find diffdrive_arduino)/ros2_control/diffbot.ros2_control.xacro" />
   <xacro:diffbot prefix="$(arg prefix)" />
-  <xacro:diffbot_ros2_control
-    name="DiffBot" prefix="$(arg prefix)" />
+  <xacro:diffbot_ros2_control name="DiffBot" prefix="$(arg prefix)" />
 </robot>

File: description/urdf/diffbot_description.urdf.xacro (robot description, xacro)
@@ -8,11 +8,13 @@
   <xacro:property name="base_width" value="0.145" />
   <xacro:property name="base_length" value="0.168" />
-  <xacro:property name="base_height" value="0.02" />
+  <xacro:property name="base_height" value="0.065" />
   <xacro:property name="wheel_mass" value="0.3" /> <!-- arbitrary value for wheel mass -->
   <xacro:property name="wheel_len" value="0.014" />
   <xacro:property name="wheel_radius" value="0.0475" />
+  <xacro:property name="wheel_xoff" value="0.054"/>
+  <xacro:property name="wheel_zoff" value="-0.005"/>
   <xacro:property name="caster_wheel_mass" value="0.1" /> <!-- arbitrary value for caster wheel mass -->
   <xacro:property name="caster_wheel_radius" value="0.015" />
-  <xacro:property name="z_offset" value="-${base_height/2}" /> <!-- Space btw top of beam and the each joint -->
+  <xacro:property name="caster_xoff" value="-0.06"/>
   <!-- Base Link -->
   <link name="${prefix}base_link">
@@ -42,5 +44,5 @@
       <parent link="${prefix}base_link"/>
       <child link="${prefix}left_wheel"/>
-      <origin xyz="0 -${base_width/2} ${z_offset}" rpy="0 0 0"/>
+      <origin xyz="${wheel_xoff} -${base_width/2} ${wheel_zoff}" rpy="0 0 0"/>
       <axis xyz="0 1 0"/>
       <dynamics damping="0.2"/>
@@ -73,5 +75,5 @@
       <parent link="${prefix}base_link"/>
       <child link="${prefix}right_wheel"/>
-      <origin xyz="0 ${base_width/2} ${z_offset}" rpy="0 0 0"/>
+      <origin xyz="${wheel_xoff} ${base_width/2} ${wheel_zoff}" rpy="0 0 0"/>
       <axis xyz="0 1 0"/>
       <dynamics damping="0.2"/>
@@ -101,11 +103,11 @@
         </inertial>
       </link>
-    <joint name="${prefix}caster_rear_wheel_joint" type="fixed">
+    <joint name="${prefix}caster_wheel_joint" type="fixed">
       <parent link="${prefix}base_link"/>
-      <child link="${prefix}caster_rear_wheel"/>
-      <origin xyz="${-base_width/2 + caster_wheel_radius} 0 ${z_offset}" rpy="0 0 0"/>
+      <child link="${prefix}caster_wheel"/>
+      <origin xyz="${caster_xoff} 0 ${-(base_height/2)}" rpy="0 0 0"/>
     </joint>
     <!-- caster rear wheel Link -->
-    <link name="${prefix}caster_rear_wheel">
+    <link name="${prefix}caster_wheel">
       <collision>
         <origin xyz="0 0 0" rpy="0 0 0"/>

File: description/urdf/lidar.xacro (robot description, xacro)
@@ -4,5 +4,5 @@
         <parent link="base_link"/>
         <child link="laser_frame"/>
-        <origin xyz="0.05 0 0.03" rpy="0 0 0"/>
+        <origin xyz="0 0 0.12" rpy="0 0 0"/>
     </joint>
     <link name="laser_frame">
